Commit message: arm part 8 collision inertia fixed

File: src/my_robot_description/urdf/far_common_properties.xml.xacro (robot description, xacro)
@@ -43,7 +43,4 @@
     <xacro:property name="controller_width" value="0.04" />
     <xacro:property name="controller_height" value="0.1" />
-    <xacro:property name="arm_base_length" value="0.1" />
-    <xacro:property name="arm_base_width" value="0.1" />
-    <xacro:property name="arm_base_height" value="0.03" />
     <xacro:property name="arm_base_length" value="0.1" />
     <xacro:property name="arm_base_width" value="0.1" />

File: src/my_robot_description/urdf/main_arm_units.xml.xacro (robot description, xacro)
@@ -162,12 +162,12 @@
                 <material name="link_common_color" />
             </visual>
-            <!-- <collision>
-                <geometry>
-                    <box size="${arm_link_3_length} ${arm_link_3_width} ${arm_link_3_height}" />
-                </geometry>
-                <origin xyz="0 0 ${arm_link_3_height/2+arm_joint_3_radius}" rpy="0 0 0" />
-            </collision>
-            <xacro:box_inertia m="1.0" x="${arm_link_3_length}" y="${arm_link_3_width}" z="${arm_link_3_height}"
-                            o_xyz="0 0 ${arm_link_3_height/2+arm_joint_3_radius}" o_rpy="0 0 0" /> -->
+            <collision>
+                <geometry>
+                    <box size="${0.01} ${0.01} ${arm_joint_2_radius+arm_link_1_height+arm_joint_1_length}" />
+                </geometry>
+                <origin xyz="0 0 ${arm_joint_2_radius/2+arm_link_1_height/2+arm_joint_1_length/2}" rpy="0 0 0" />
+            </collision>
+            <xacro:box_inertia m="0.1" x="0.01" y="0.01" z="${arm_joint_2_radius+arm_link_1_height+arm_joint_1_length}"
+                            o_xyz="0 0 ${arm_joint_2_radius/2+arm_link_1_height/2+arm_joint_1_length/2}" o_rpy="0 0 0" />
         </link>
     </xacro:macro>

Commit message: panorama camera

File: src/my_robot_description/urdf/far_common_properties.xml.xacro (robot description, xacro)
@@ -36,4 +36,7 @@
     <material name="controller_color">
         <color rgba="0.1 0.8 0.8 1" />
+    </material>
+    <material name="camera_color">
+        <color rgba="0.1 0.1 0.1 1" />
     </material>
     <xacro:property name="battery_length" value="0.08" />
@@ -83,4 +86,9 @@
     <xacro:property name="gripper_link_width" value="0.04" />
     <xacro:property name="gripper_link_height" value="0.05" />
+     <xacro:property name="camera_length" value="0.02" />
+     <xacro:property name="camera_width" value="0.02" />
+     <xacro:property name="camera_height" value="0.02" />
+     <xacro:property name="camera_mass" value="0.02" />
+     <xacro:property name="camera_optical_size" value="0.005" />
     <xacro:macro name="box_inertia" params="m x y z o_xyz o_rpy">
         <inertial>

File: src/my_robot_description/urdf/four_arm_robot.xml.xacro (robot description, xacro)
@@ -5,4 +5,5 @@
     <xacro:include filename="mobile_base_part.xml.xacro" />
     <xacro:include filename="branch_arm_unit.xml.xacro" />
+    <xacro:include filename="unit_camera.xml.xacro" />
     <link name="base_footprint" />
     <joint name="base_joint" type="fixed">
@@ -33,3 +34,18 @@
     </xacro:macro>
     <xacro:branch_joint prefix="4" />
+    <xacro:macro name="camera_mount_joint" params="prefix">
+        <joint name="camera_joint_${prefix}" type="fixed">
+            <parent link="arm_base_link_${prefix}" />
+            <child link="camera_link_${prefix}" />
+            <origin xyz="-${arm_base_length/2-camera_length/2} ${arm_base_width/2-camera_width/2} ${arm_base_height/2+camera_height/2}" rpy="0 0 -${pi/4.0}" />
+        </joint>
+    </xacro:macro>
+    <xacro:camera_unit prefix="1" />
+    <xacro:camera_mount_joint prefix="1" />
+    <xacro:camera_unit prefix="2" />
+    <xacro:camera_mount_joint prefix="2" />
+    <xacro:camera_unit prefix="3" />
+    <xacro:camera_mount_joint prefix="3" />
+    <xacro:camera_unit prefix="4" />
+    <xacro:camera_mount_joint prefix="4" />
 </robot>
