Commit message: rviz display and joint state set

File: src/my_robot_description/urdf/far_common_properties.xml.xacro (robot description, xacro)
@@ -50,5 +50,5 @@
     <xacro:property name="arm_base_height" value="0.03" />
     <xacro:property name="veer_length" value="0.04" />
-    <xacro:property name="veer_width" value="0.04" />
+    <xacro:property name="veer_width" value="0.02" />
     <xacro:property name="veer_height" value="0.01" />
     <xacro:property name="wheel_radius" value="0.04" />

File: src/my_robot_description/urdf/four_arm_robot.xml.xacro (robot description, xacro)
@@ -20,6 +20,6 @@
             <origin xyz="0 0 -${arm_base_height/2}" rpy="0 0 0" />
             <axis xyz="0 0 1"/>
-            <limit lower="${-pi}" upper="${pi}" effort="10" velocity="1.0"/>
-            <dynamics friction="100.0" damping="0.3" />
+            <limit lower="${-pi}" upper="${pi}" effort="100" velocity="1.0"/>
+            <dynamics friction="0.1" damping="0.1" />
         </joint>
     </xacro:macro>

File: src/my_robot_description/urdf/mobile_base_part.xml.xacro (robot description, xacro)
@@ -31,7 +31,7 @@
             <collision>
                 <geometry>
-                    <sphere radius="0.1" />
+                    <cylinder radius="${wheel_radius}" length="${wheel_length}" />
                 </geometry>
-                <origin xyz="0 0 0" rpy="0 0 0" />
+                <origin xyz="0 0 0" rpy="${pi / 2.0} 0 0" />
             </collision>
             <xacro:cylinder_inertia m="1.0" r="${wheel_radius}" l="${wheel_length}"

File: src/my_robot_description/urdf/unit_camera.xml.xacro (robot description, xacro)
@@ -55,5 +55,5 @@
                 </camera>
                 <always_on>1</always_on>
-                <update_rate>1</update_rate>
+                <update_rate>5</update_rate>
                 <visualize>true</visualize>
                 <topic>camera_${prefix}/image_raw</topic>
