Commit message: gazebo world

File: src/my_robot_description/urdf/four_arm_robot.xml.xacro (robot description, xacro)
@@ -18,4 +18,5 @@
             <axis xyz="0 0 1"/>
             <limit lower="-0.8" upper="0.8" effort="10" velocity="1.0"/>
+            <dynamics friction="100.0" damping="0.3" />
         </joint>
     </xacro:macro>

File: src/my_robot_description/urdf/main_arm_units.xml.xacro (robot description, xacro)
@@ -215,5 +215,5 @@
             <axis xyz="0 0 1" />
             <limit lower="-3.14" upper="3.14" effort="100" velocity="100" />
-            <dynamics friction="0.3" damping="0.3" />
+            <dynamics friction="100.0" damping="0.3" />
         </joint>
     </xacro:macro>
@@ -232,5 +232,5 @@
             <axis xyz="0 1 0" />
             <limit lower="-2.35" upper="2.35" effort="100" velocity="100" />
-            <dynamics friction="0.3" damping="0.3" />
+            <dynamics friction="100.0" damping="0.3" />
         </joint>
     </xacro:macro>
@@ -249,5 +249,5 @@
             <axis xyz="0 1 0" />
             <limit lower="-2.35" upper="2.35" effort="100" velocity="100" />
-            <dynamics friction="0.3" damping="0.3" />
+            <dynamics friction="100.0" damping="0.3" />
         </joint>
     </xacro:macro>
@@ -266,5 +266,5 @@
             <axis xyz="0 1 0" />
             <limit lower="-2.35" upper="2.35" effort="100" velocity="100" />
-            <dynamics friction="0.3" damping="0.3" />
+            <dynamics friction="100.0" damping="0.3" />
         </joint>
     </xacro:macro>
@@ -352,5 +352,5 @@
                 <origin xyz="0 0 ${controller_height/2+arm_joint_2_radius}" rpy="0 0 0" />
             </collision>
-            <xacro:box_inertia m="1.0" x="${controller_length}" y="${controller_width}" z="${controller_height}"
+            <xacro:box_inertia m="2.0" x="${controller_length}" y="${controller_width}" z="${controller_height}"
                             o_xyz="0 0 ${arm_link_2_height/2+arm_joint_2_radius}" o_rpy="0 0 0" />
         </link>

Commit message: fix problem sdf sensor

File: src/my_robot_description/urdf/four_arm_robot.xml.xacro (robot description, xacro)
@@ -38,5 +38,5 @@
             <parent link="arm_base_link_${prefix}" />
             <child link="camera_link_${prefix}" />
-            <origin xyz="-${arm_base_length/2-camera_length/2} ${arm_base_width/2-camera_width/2} ${arm_base_height/2+camera_height/2}" rpy="0 0 -${pi/4.0}" />
+            <origin xyz="-${arm_base_length/2-camera_length/2} ${arm_base_width/2-camera_width/2} ${arm_base_height/2+camera_height/2}" rpy="0 0 ${pi*3.0/4.0}" />
         </joint>
     </xacro:macro>
