Commit message: gazebo controller

File: src/my_robot_description/urdf/four_arm_robot.xml.xacro (robot description, xacro)
@@ -7,4 +7,5 @@
     <xacro:include filename="unit_camera.xml.xacro" />
     <xacro:include filename="stereo_camera.xml.xacro" />
+    <xacro:include filename="my_robot.ros2_control.xacro" />
     <link name="base_footprint" />
     <joint name="base_joint" type="fixed">
@@ -19,5 +20,5 @@
             <origin xyz="0 0 -${arm_base_height/2}" rpy="0 0 0" />
             <axis xyz="0 0 1"/>
-            <limit lower="-0.8" upper="0.8" effort="10" velocity="1.0"/>
+            <limit lower="${-pi}" upper="${pi}" effort="10" velocity="1.0"/>
             <dynamics friction="100.0" damping="0.3" />
         </joint>
@@ -50,3 +51,8 @@
     <xacro:camera_unit prefix="4" />
     <xacro:camera_mount_joint prefix="4" />
+    <gazebo>
+        <plugin filename="libgz_ros2_control-system.so" name="gz_ros2_control::GazeboSimROS2ControlPlugin">
+            <parameters>$(find my_robot_bringup)/config/ros2_controllers.yaml</parameters>
+        </plugin>
+    </gazebo>
 </robot>

File: src/my_robot_description/urdf/stereo_camera.xml.xacro (robot description, xacro)
@@ -34,10 +34,10 @@
         <parent link="branch_arm_link_4" />
         <child link="camera_link_5" />
-        <origin xyz="${(branch_arm_link_length)/2.0} ${branch_arm_link_width*2} ${branch_arm_link_height/2.0}" rpy="-${pi/2.0} 0 0" />
+        <origin xyz="${(branch_arm_link_length)/2.0} ${branch_arm_link_width*2} ${branch_arm_link_height/2.0}" rpy="${pi} ${-pi/4.0} 0" />
     </joint>
     <joint name="base_camera_joint_6" type="fixed">
         <parent link="branch_arm_link_4" />
         <child link="camera_link_6" />
-        <origin xyz="${(branch_arm_link_length)/2.0} ${-branch_arm_link_width*2} ${branch_arm_link_height/2.0}" rpy="-${pi/2.0} 0 0" />
+        <origin xyz="${(branch_arm_link_length)/2.0} ${-branch_arm_link_width*2} ${branch_arm_link_height/2.0}" rpy="${pi} ${-pi/4.0} 0" />
     </joint>
     <link name="camera_link_optical_5" />
@@ -75,5 +75,5 @@
             </camera>
             <always_on>1</always_on>
-            <update_rate>20</update_rate>
+            <update_rate>5</update_rate>
             <visualize>true</visualize>
             <topic>camera_5/image_raw</topic>
@@ -102,5 +102,5 @@
             </camera>
             <always_on>1</always_on>
-            <update_rate>20</update_rate>
+            <update_rate>5</update_rate>
             <visualize>true</visualize>
             <topic>camera_6/image_raw</topic>

Commit message: urdf error fixed

File: src/my_robot_description/urdf/four_arm_robot.xml.xacro (robot description, xacro)
@@ -14,5 +14,5 @@
         <origin xyz="0 0 ${wheel_radius*2+veer_height+arm_base_height/2}" rpy="0 0 0" />
     </joint>
-    <xacro:macro name="group_joint" params="prefix">
+    <xacro:macro name="arm_veer_joint" params="prefix">
         <joint name="arm_veer_joint_${prefix}" type="revolute">
             <parent link="arm_base_link_${prefix}" />
@@ -24,8 +24,8 @@
         </joint>
     </xacro:macro>
-    <xacro:group_joint prefix="1" />
-    <xacro:group_joint prefix="2" />
-    <xacro:group_joint prefix="3" />
-    <xacro:group_joint prefix="4" />
+    <xacro:arm_veer_joint prefix="1" />
+    <xacro:arm_veer_joint prefix="2" />
+    <xacro:arm_veer_joint prefix="3" />
+    <xacro:arm_veer_joint prefix="4" />
     <xacro:macro name="branch_joint" params="prefix">
         <joint name="branch_joint_${prefix}" type="fixed">
