Commit message: stereo camera

File: src/my_robot_description/urdf/branch_arm_unit.xml.xacro (robot description, xacro)
@@ -22,4 +22,23 @@
     <xacro:macro name="branch_connecter" params="prefix">
         <link name="branch_connecter_${prefix}">
+            <visual>
+                <geometry>
+                    <box size="${connecter_link_length} ${connecter_link_width} ${connecter_link_height}" />
+                </geometry>
+                <origin xyz="0 0 ${connecter_link_height/2}" rpy="0 0 0" />
+                <material name="branch_link_color" />
+            </visual>
+            <collision>
+                <geometry>
+                    <box size="${connecter_link_length} ${connecter_link_width} ${connecter_link_height}" />
+                </geometry>
+                <origin xyz="0 0 ${connecter_link_height/2}" rpy="0 0 0" />
+            </collision>
+            <xacro:box_inertia m="0.5" x="${connecter_link_length}" y="${connecter_link_width}" z="${connecter_link_height}"
+                            o_xyz="0 0 ${connecter_link_height/2}" o_rpy="0 0 0" />
+        </link>
+    </xacro:macro>
+    <xacro:macro name="camera_connecter" params="prefix">
+        <link name="camera_connecter_${prefix}">
             <visual>
                 <geometry>

File: src/my_robot_description/urdf/four_arm_robot.xml.xacro (robot description, xacro)
@@ -6,4 +6,5 @@
     <xacro:include filename="branch_arm_unit.xml.xacro" />
     <xacro:include filename="unit_camera.xml.xacro" />
+    <xacro:include filename="stereo_camera.xml.xacro" />
     <link name="base_footprint" />
     <joint name="base_joint" type="fixed">
@@ -30,5 +31,5 @@
             <parent link="arm_part_6_${prefix}" />
             <child link="branch_arm_link_${prefix}" />
-            <origin xyz="0 ${arm_link_3_width/2+branch_arm_link_width/2} ${arm_link_3_height+arm_joint_3_radius}" rpy="0 0 0" />
+            <origin xyz="0 ${arm_link_3_width/2+branch_arm_link_width/2+0.05} ${arm_link_3_height+arm_joint_3_radius}" rpy="0 0 0" />
         </joint>
     </xacro:macro>

File: src/my_robot_description/urdf/unit_camera.xml.xacro (robot description, xacro)
@@ -43,6 +43,6 @@
                     </image>
                     <clip>
-                        <near>0.05</near>
-                        <far>8.0</far>
+                        <near>0.3</near>
+                        <far>16.0</far>
                     </clip>
                     <noise>
