Commit message: arm urdf fix

File: src/my_robot_description/urdf/main_arm_units.xml.xacro (robot description, xacro)
@@ -150,5 +150,5 @@
             </collision>
             <xacro:cylinder_inertia m="2.0" r="${arm_joint_4_radius}" l="${arm_joint_4_length}"
-                                o_xyz="0 0 0" o_rpy="${pi / 4.0} 0 0"/>
+                                o_xyz="0 0 0" o_rpy="${pi / 2.0} 0 0"/>
         </link>
     </xacro:macro>
@@ -215,5 +215,5 @@
             <axis xyz="0 0 1" />
             <limit lower="-3.14" upper="3.14" effort="100" velocity="100" />
-            <dynamics friction="100.0" damping="0.3" />
+            <dynamics friction="0.1" damping="0.1" />
         </joint>
     </xacro:macro>
@@ -232,5 +232,5 @@
             <axis xyz="0 1 0" />
             <limit lower="-2.35" upper="2.35" effort="100" velocity="100" />
-            <dynamics friction="100.0" damping="0.3" />
+            <dynamics friction="0.1" damping="0.1" />
         </joint>
     </xacro:macro>
@@ -249,5 +249,5 @@
             <axis xyz="0 1 0" />
             <limit lower="-2.35" upper="2.35" effort="100" velocity="100" />
-            <dynamics friction="100.0" damping="0.3" />
+            <dynamics friction="0.1" damping="0.1" />
         </joint>
     </xacro:macro>
@@ -266,5 +266,5 @@
             <axis xyz="0 1 0" />
             <limit lower="-2.35" upper="2.35" effort="100" velocity="100" />
-            <dynamics friction="100.0" damping="0.3" />
+            <dynamics friction="0.1" damping="0.1" />
         </joint>
     </xacro:macro>
